Commit message: update urdf

File: assets/aubo_description/urdf/aubo_iS10.urdf (robot description, URDF)
Before this commit: robot aubo_iS10, 8 links, 7 joints
Links:
- link base_link: geometry collision mesh filename=package://aubo_description/meshes/aubo_iS10/collision/link0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; visual mesh filename=package://aubo_description/meshes/aubo_iS10/collision/link0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
- link foreArm_Link: geometry collision mesh filename=package://aubo_description/meshes/aubo_iS10/collision/link3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; visual mesh filename=package://aubo_description/meshes/aubo_iS10/collision/link3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
- link shoulder_Link: geometry collision mesh filename=package://aubo_description/meshes/aubo_iS10/collision/link1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; visual mesh filename=package://aubo_description/meshes/aubo_iS10/collision/link1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
- link upperArm_Link: geometry collision mesh filename=package://aubo_description/meshes/aubo_iS10/collision/link2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; visual mesh filename=package://aubo_description/meshes/aubo_iS10/collision/link2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
- link wrist1_Link: geometry collision mesh filename=package://aubo_description/meshes/aubo_iS10/collision/link4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; visual mesh filename=package://aubo_description/meshes/aubo_iS10/collision/link4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
- link wrist2_Link: geometry collision mesh filename=package://aubo_description/meshes/aubo_iS10/collision/link5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; visual mesh filename=package://aubo_description/meshes/aubo_iS10/collision/link5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
- link wrist3_Link: geometry collision mesh filename=package://aubo_description/meshes/aubo_iS10/collision/link6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; visual mesh filename=package://aubo_description/meshes/aubo_iS10/collision/link6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
